File: Duet2/Duet2lite/Stepper_Drv.sch (KiCad schematic (older format))
At the start: 110 parts, among them U10 74HC125, U13 74HC32, U5 TMC2660, U6 TMC2660, U7 TMC2660, U8 TMC2660, U9 TMC2660

Commit message: removed stepper drivers from the schematic
Parts:
- removed C100, C20, C21, C30, C31: 0u47, complib:C_0603, symbol DuetWifi:C_SMALL
- removed C101, C75, C76, C77, C78: 1u 50V, complib:C_0603, symbol DuetWifi:C_SMALL
- removed C102, C22, C23, C32, C33: 100u 35V, complib:C_ELEC_6.3x7.7, symbol DuetWifi:C_POL
- removed C103, C24, C25, C34, C35: 0u1 50V, complib:C_0603, symbol DuetWifi:C_SMALL
- removed C104, C26, C27, C36, C37: 0u1, complib:C_0603, symbol DuetWifi:C_SMALL
- removed C105, C110, C14, C15, C28, C29, C38, C39, C56, C57: 0u01 X7R 10% 50V, complib:C_0603, symbol DuetWifi:C_SMALL
- removed C106, C107, C108, C109, C113, C114, C115, C116, C117, C118, C119, C120, C121, C122, C123, C85, C86, C87, C88, C89: 1n >50V, complib:C_0603, symbol DuetWifi:C_SMALL
- removed R26, R27, R28, R29, R38, R39, R40, R41, R89, R90: 22R, complib:R_0603, symbol DuetWifi:R_SMALL
- removed R32, R33, R34, R35, R44, R45, R46, R47, R93, R94: 0R051, complib:R_1206, symbol DuetWifi:R_SMALL
- removed U5, U6, U7, U8, U9: TMC2660, FE Footprints:TMC2660, symbol DuetWifi:TMC2660
- added J?: XAxisStepper, symbol Duet2Lite:Conn_01x10
- added J?: YAxisStepper, symbol Duet2Lite:Conn_01x10
- added J?: ZAxisStepper, symbol Duet2Lite:Conn_01x10
- added J?: E0Stepper, symbol Duet2Lite:Conn_01x10
- added J?: E1Stepper, symbol Duet2Lite:Conn_01x10
- D22, D23, D24: symbol DuetWifi:DIODESCH -> Duet2Lite:BAT54C
Connections:
- net +3.3V: now also D22.3, D23.3, D24.3, J?.1 (Pin_1), J?.1 (Pin_1), J?.1 (Pin_1), J?.1 (Pin_1), J?.1 (Pin_1)
- net E0_DIR: now also J?.3 (Pin_3)
- net E0_EN: now also J?.4 (Pin_4)
- net E0_STEP: now also J?.2 (Pin_2)
- net E0_STOP: now also D23.2
- net E1_DIR: now also J?.3 (Pin_3)
- net E1_EN: now also J?.4 (Pin_4)
- net E1_STEP: now also J?.2 (Pin_2)
- net E1_STOP: now also D24.1
- net ENN: now also J?.8 (Pin_8), J?.8 (Pin_8), J?.8 (Pin_8), J?.8 (Pin_8), J?.8 (Pin_8)
- net GND: now also J?.10 (Pin_10), J?.10 (Pin_10), J?.10 (Pin_10), J?.10 (Pin_10), J?.10 (Pin_10)
- net SG_TST_E0: now also J?.9 (Pin_9)
- net SG_TST_E1: now also J?.9 (Pin_9)
- net SG_TST_X: now also J?.9 (Pin_9)
- net SG_TST_Y: now also J?.9 (Pin_9)
- net SG_TST_Z: now also J?.9 (Pin_9)
- net SPI1_MISO: now also J?.7 (Pin_7), J?.7 (Pin_7), J?.7 (Pin_7), J?.7 (Pin_7), J?.7 (Pin_7)
- net SPI1_MOSI_BUFF: now also J?.6 (Pin_6), J?.6 (Pin_6), J?.6 (Pin_6), J?.6 (Pin_6), J?.6 (Pin_6)
- net SPI1_SCK_BUFF: now also J?.5 (Pin_5), J?.5 (Pin_5), J?.5 (Pin_5), J?.5 (Pin_5), J?.5 (Pin_5)
- net X_DIR: now also J?.3 (Pin_3)
- net X_EN: now also J?.4 (Pin_4)
- net X_STEP: now also J?.2 (Pin_2)
- net X_STOP: now also D23.1
- net Y_DIR: now also J?.3 (Pin_3)
- net Y_EN: now also J?.4 (Pin_4)
- net Y_STEP: now also J?.2 (Pin_2)
- net Y_STOP: now also D22.1
- net Z_DIR: now also J?.3 (Pin_3)
- net Z_EN: now also J?.4 (Pin_4)
- net Z_PROBE_MCU: now also D24.2
- net Z_STEP: now also J?.2 (Pin_2)
- net Z_STOP: now also D22.2
- no-connect marks 16 -> 1
Other:
- note removed: "C20 between pin 13 and 17"
- note removed: "C21 between pin 13 and 17"
- note removed: "C30 between pin 13 and 17"
